File: Plate/v.4.0.1_steady/keyplate/keyplate.kicad_pcb (KiCad board)
At the start: 2 copper layers, 284.7 x 94.7 mm, 3 parts

Commit message: Created rev2
Other:
- outline, holes or cut-outs redrawn
- board text added: "#Jones_kbd Unofficial Keyplate {dblquote}Steady{dblquote} rev.2 @tamano"
- board text removed: "#Jones_kbd Unofficial Keyplate {dblquote}Steady{dblquote} rev.1, @tamano"
